File: switch_matrix.kicad_sch (KiCad schematic)
At the start: 136 parts

Commit message: Finalized hardware Ver 1 release
Other:
- company: (none) -> HW-tinkerers
Changed lines of the file:
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@@
 (kicad_sch (version 20230121) (generator eeschema)
   (paper "A4")
+  (title_block
+    (date "2024-02-17")
+    (company "HW-tinkerers")
+  )
   (junction (at 214.63 114.3) (diameter 0) (color 0 0 0 0)
   )
