File: Keyboard_60%.kicad_pcb (KiCad board)
At the start: 2 copper layers, 284.7 x 94.2 mm, 215 parts, among them J1 JST-4-pin, J3 Prog_conn, J4 TYPE-C-31-M12_13, J5 Tag connect TC2030-CTX, SW1 MK-12C02-G025, SW2 Reset Switch, U1 BQ24074RGTR, U3 nRF52840-QIAA-R/nRF52833-QIAA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, U4 TPD4E05U06DQAR, Y1 32MHz, Y2 32.768kHz

Commit message: Exported edge cuts as footprint and set grid origin
Parts:
- removed the G*** at (136.0, 38.3)
- removed H1, H2, H3, H4: MountingHole, keyboard:salvation_mounting_holes
- removed H5, H6: MountingHole, keyboard:PKRHSL
- removed R19, R20, R21, R22, R23: 10k, keyboard:R_0402_1005Metric
- removed REF**: OSHW-Logo, keyboard:OSHW-Logo
- removed SW1: MK-12C02-G025, keyboard:SPDT
- added S2: ~, keyboard:Keybaord_outline_edgecuts, F.Cu at (214.3, 152.7)
- R3: value 1k2 -> 8k2
- moved D10 399.5 mm to (517.3, -104.7)
- moved D11 399.5 mm to (536.3, -104.7)
- moved D12 399.5 mm to (571.3, -104.7)
- moved D13 399.5 mm to (574.3, -104.7)
- moved D14 399.5 mm to (593.8, -104.7)
- moved D15 399.5 mm to (612.8, -104.7)
- moved D17 399.5 mm to (654.3, -101.3)
- moved D31 399.5 mm to (650.6, -92.3)
- moved D39 399.5 mm to (532.1, -67.2)
- moved D54 399.5 mm to (580.0, -48.1)
- moved D55 399.5 mm to (599.1, -48.2)
- moved D56 399.5 mm to (624.1, -48.1)
- moved D62 399.5 mm to (578.3, -33.5)
- moved AE1 399.5 mm to (389.3, -79.8)
- moved C1 399.5 mm to (429.8, -77.4)
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Connections:
- C1 pad 1: /USB and Power management/CHG_IN -> /VBUS
- D10 pad 1: /switch_matrix/ROW0 -> /ROW0
- D11 pad 1: /switch_matrix/ROW0 -> /ROW0
- D12 pad 1: /switch_matrix/ROW0 -> /ROW0
- D13 pad 1: /switch_matrix/ROW0 -> /ROW0
- D14 pad 1: /switch_matrix/ROW0 -> /ROW0
- D15 pad 1: /switch_matrix/ROW0 -> /ROW0
- D16 pad 1: /switch_matrix/ROW0 -> /ROW0
- D17 pad 1: /switch_matrix/ROW0 -> /ROW0
- D18 pad 1: /switch_matrix/ROW1 -> /ROW1
- D19 pad 1: /switch_matrix/ROW1 -> /ROW1
- D20 pad 1: /switch_matrix/ROW1 -> /ROW1
- D21 pad 1: /switch_matrix/ROW1 -> /ROW1
- D22 pad 1: /switch_matrix/ROW1 -> /ROW1
- D23 pad 1: /switch_matrix/ROW1 -> /ROW1
- D24 pad 1: /switch_matrix/ROW1 -> /ROW1
- D25 pad 1: /switch_matrix/ROW1 -> /ROW1
- D26 pad 1: /switch_matrix/ROW1 -> /ROW1
- D27 pad 1: /switch_matrix/ROW1 -> /ROW1
- D28 pad 1: /switch_matrix/ROW1 -> /ROW1
- D29 pad 1: /switch_matrix/ROW1 -> /ROW1
- D3 pad 1: /switch_matrix/ROW0 -> /ROW0
- D30 pad 1: /switch_matrix/ROW1 -> /ROW1
- D31 pad 1: /switch_matrix/ROW1 -> /ROW1
- D32 pad 1: /switch_matrix/ROW2 -> /ROW2
- D33 pad 1: /switch_matrix/ROW2 -> /ROW2
- D34 pad 1: /switch_matrix/ROW2 -> /ROW2
- D35 pad 1: /switch_matrix/ROW2 -> /ROW2
- D36 pad 1: /switch_matrix/ROW2 -> /ROW2
- D37 pad 1: /switch_matrix/ROW2 -> /ROW2
- D38 pad 1: /switch_matrix/ROW2 -> /ROW2
- D39 pad 1: /switch_matrix/ROW2 -> /ROW2
- D4 pad 1: /switch_matrix/ROW0 -> /ROW0
- D40 pad 1: /switch_matrix/ROW2 -> /ROW2
- D41 pad 1: /switch_matrix/ROW2 -> /ROW2
- D42 pad 1: /switch_matrix/ROW2 -> /ROW2
- D43 pad 1: /switch_matrix/ROW2 -> /ROW2
- D44 pad 1: /switch_matrix/ROW2 -> /ROW2
- D45 pad 1: /switch_matrix/ROW3 -> /ROW3
- D46 pad 1: /switch_matrix/ROW3 -> /ROW3
- D47 pad 1: /switch_matrix/ROW3 -> /ROW3
- D48 pad 1: /switch_matrix/ROW3 -> /ROW3
- D49 pad 1: /switch_matrix/ROW3 -> /ROW3
- D5 pad 1: /switch_matrix/ROW0 -> /ROW0
- D50 pad 1: /switch_matrix/ROW3 -> /ROW3
- D51 pad 1: /switch_matrix/ROW3 -> /ROW3
- D52 pad 1: /switch_matrix/ROW3 -> /ROW3
- D53 pad 1: /switch_matrix/ROW3 -> /ROW3
- D54 pad 1: /switch_matrix/ROW3 -> /ROW3
- D55 pad 1: /switch_matrix/ROW3 -> /ROW3
- D56 pad 1: /switch_matrix/ROW3 -> /ROW3
- D57 pad 1: /switch_matrix/ROW3 -> /ROW3
- D58 pad 1: /switch_matrix/ROW4 -> /ROW4
- D59 pad 1: /switch_matrix/ROW4 -> /ROW4
- D6 pad 1: /switch_matrix/ROW0 -> /ROW0
- D60 pad 1: /switch_matrix/ROW4 -> /ROW4
- D61 pad 1: /switch_matrix/ROW4 -> /ROW4
- D62 pad 1: /switch_matrix/ROW4 -> /ROW4
- D63 pad 1: /switch_matrix/ROW4 -> /ROW4
- D64 pad 1: /switch_matrix/ROW4 -> /ROW4
- D65 pad 1: /switch_matrix/ROW4 -> /ROW4
- D7 pad 1: /switch_matrix/ROW0 -> /ROW0
- D8 pad 1: /switch_matrix/ROW0 -> /ROW0
- D9 pad 1: /switch_matrix/ROW0 -> /ROW0
- J1 pad 1: /USB and Power management/VBUS -> /VBUS
- J4 pad A4: /USB and Power management/VBUS -> /VBUS
- J4 pad B4: /USB and Power management/VBUS -> /VDDH
- R1 pad 1: /VBUS -> /VDDH
- R2 pad 1: /VBUS -> /VDDH
- U1 pad 10: /VBUS -> /VDDH
- U1 pad 11: /VBUS -> /VDDH
- U1 pad 13: /USB and Power management/CHG_IN -> /VBUS
- U1 pad 5: /VBUS -> /VDDH
- U3 pad Y2: /VBUS -> /VDDH
Routing:
- net /ROW3: track 39.3 -> 343.6 mm
- net /switch_matrix/ROW3: track 304.3 -> 0.00 mm
- net /ROW4: track 62.9 -> 349.2 mm
- net /switch_matrix/ROW4: track 286.3 -> 0.00 mm
- net /ROW0: track 26.0 -> 309.4 mm
- net /switch_matrix/ROW0: track 283.4 -> 0.00 mm
- net /ROW2: track 28.4 -> 311.7 mm, vias 2 -> 4
- net /switch_matrix/ROW2: track 283.2 -> 0.00 mm, vias 2 -> 0
- net /switch_matrix/ROW1: track 267.4 -> 0.00 mm, vias 2 -> 0
- net /ROW1: track 17.7 -> 285.1 mm, vias 2 -> 4
- net /VBUS: track 65.5 -> 181.6 mm, vias 7 -> 13
- net /USB and Power management/VBUS: track 115.9 -> 0.00 mm, vias 4 -> 0
- net /USB and Power management/CHG_IN: track 28.5 -> 0.00 mm, vias 2 -> 0
- net /COL1: track 138.7 -> 126.4 mm
- net Net-(D4-A): track 11.7 -> 0.00 mm
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Other:
- outline, holes or cut-outs redrawn

Commit message: Completed routing for rows
Parts:
- removed kibuzzard-64CB1AC3: G***, kibuzzard-64CB1AC3
- moved D59 385.7 mm to (112.0, 190.5)
- moved D12 383.5 mm to (257.0, 115.0)
- moved D9 383.4 mm to (200.0, 115.0)
- moved D62 380.3 mm to (271.0, 190.5), turned to 90 degrees
- moved D31 379.9 mm to (350.0, 140.0), turned to 0 degrees
- moved D21 378.0 mm to (152.0, 133.3), turned to 90 degrees
- moved D22 378.0 mm to (171.0, 133.3), turned to 90 degrees
- moved D23 377.9 mm to (190.0, 133.3), turned to 90 degrees
- moved D30 377.6 mm to (324.0, 133.3), turned to 90 degrees
- moved D29 377.2 mm to (305.0, 133.3), turned to 90 degrees
- moved D24 377.2 mm to (210.0, 133.3), turned to 90 degrees
- moved D25 377.2 mm to (229.0, 133.3), turned to 90 degrees
- moved D28 377.2 mm to (286.0, 133.3), turned to 90 degrees
- moved D26 377.1 mm to (248.0, 133.3), turned to 90 degrees
- moved D27 377.1 mm to (267.0, 133.3), turned to 90 degrees
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Routing:
- net /COL13: track 367.3 -> 6.02 mm, vias 2 -> 1
- net /COL12: track 341.7 -> 14.8 mm, vias 4 -> 1
- net /COL14: track 296.4 -> 9.01 mm, vias 2 -> 1
- net /COL11: track 301.5 -> 17.6 mm
- net /COL10: track 283.2 -> 15.2 mm
- net /COL9: track 243.9 -> 15.4 mm
- net /COL8: track 224.6 -> 15.4 mm
- net /COL6: track 218.6 -> 12.9 mm, vias 2 -> 1
- net /COL7: track 205.6 -> 15.9 mm
- net /VBUS: track 181.6 -> 9.23 mm, vias 13 -> 2
- net /COL5: track 166.9 -> 5.13 mm, vias 2 -> 1
- net /COL2: track 170.2 -> 13.9 mm, vias 4 -> 1
- net /COL4: track 151.6 -> 4.73 mm, vias 2 -> 1
- net /COL0: track 172.2 -> 32.7 mm, vias 4 -> 0
- net /COL3: track 135.4 -> 8.10 mm, vias 2 -> 1
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Other:
- outline, holes or cut-outs redrawn
- board text removed: "BAT + USB"
- board text removed: "ONLY"
- board text removed: "USB"

Commit message: Completed routing for columns and rows for NRF
Parts:
- moved J1 447.7 mm to (132.9, 123.0)
- moved J3 369.9 mm to (89.3, 173.0)
- moved J5 369.9 mm to (90.3, 186.1)
- moved JP1 369.9 mm to (91.1, 182.5)
- moved R10 369.9 mm to (93.5, 176.4)
- moved R11 369.9 mm to (93.5, 171.5)
- moved R12 369.9 mm to (93.6, 168.2)
- moved R13 369.9 mm to (93.2, 169.8)
- moved R18 369.9 mm to (93.6, 175.2)
- moved R8 369.9 mm to (93.1, 178.0)
- moved R9 369.9 mm to (93.1, 173.0)
- moved D58 1.61 mm to (89.4, 192.1)
- moved D45 1.54 mm to (99.4, 172.1)
Routing:
- net /COL13: track 6.02 -> 321.9 mm, vias 1 -> 2
- net /COL12: track 14.8 -> 320.1 mm, vias 1 -> 3
- net /COL14: track 9.01 -> 289.8 mm, vias 1 -> 2
- net /COL11: track 17.6 -> 297.7 mm
- net /COL10: track 15.2 -> 277.9 mm
- net /COL9: track 15.4 -> 237.9 mm
- net /COL6: track 12.9 -> 231.5 mm, vias 1 -> 4
- net /COL8: track 15.4 -> 218.5 mm
- net /COL7: track 15.9 -> 198.7 mm
- net /COL5: track 5.13 -> 164.8 mm, vias 1 -> 2
- net /COL4: track 4.73 -> 149.4 mm, vias 1 -> 2
- net /COL2: track 13.9 -> 143.3 mm, vias 1 -> 2
- net /COL3: track 8.10 -> 132.0 mm, vias 1 -> 2
- net /COL0: track 32.7 -> 154.5 mm, vias 0 -> 4
- net /COL1: track 10.5 -> 131.8 mm
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
Commit message: Added charger circuit
Parts:
- moved BT1 440.0 mm to (152.4, 159.8)
- moved C1 399.6 mm to (135.3, 147.6)
- moved R1 399.6 mm to (137.2, 154.0)
- moved R2 399.6 mm to (138.5, 154.0)
- moved R3 399.6 mm to (138.6, 147.5)
- moved R4 399.6 mm to (134.4, 149.3)
- moved D1 399.6 mm to (139.5, 157.3)
- moved D2 399.6 mm to (142.0, 157.3)
- moved R5 399.6 mm to (137.4, 147.5)
- moved TH1 399.6 mm to (140.4, 148.8)
- moved U1 399.6 mm to (137.2, 150.6)
- moved C2 399.5 mm to (140.4, 151.6)
- moved R14 396.6 mm to (144.7, 148.4)
- moved D34 9.71 mm to (146.0, 158.0), turned to 180 degrees
- moved D35 9.71 mm to (165.0, 158.0), turned to 180 degrees
Routing:
- net /VBATT_nRF: track 8.48 -> 47.8 mm, vias 2 -> 4
- net /USB and Power management/V_BATT: track 7.03 -> 21.5 mm
- net /VDDH: track 7.53 -> 15.3 mm, vias 0 -> 2
- net /ROW2: track 324.7 -> 318.0 mm
- net /VBUS: track 9.23 -> 5.97 mm, vias 2 -> 0
- net /COL6: track 231.5 -> 228.4 mm, vias 4 -> 5
- net /COL2: track 143.3 -> 146.2 mm
- net /COL3: track 132.0 -> 134.8 mm
- net /USB_D-: track 19.3 -> 21.7 mm
- net /USB_D+: track 20.3 -> 22.4 mm
- net Net-(D35-A): track 6.18 -> 7.92 mm
- net Net-(D34-A): track 6.13 -> 7.78 mm

Commit message: Solved all DRC and updated Versioning
Parts:
- removed the G*** at (481.0, 91.5)
- added S1: Open Hardware, keyboard:OSHW-Logo, F.Cu at (209.7, 142.7)
- added S3: ~, keyboard:BLE-symbol, F.Cu at (233.6, 145.2)
- added S4: ~, keyboard:ZMK_logo, F.Cu at (222.5, 143.4)
- moved SW2 467.0 mm to (121.2, 172.8)
- moved G*** 320.8 mm to (194.9, 191.6)
- moved G*** 292.0 mm to (252.0, 194.4)
- moved G*** 292.0 mm to (254.3, 185.7)
- moved D2 3.01 mm to (139.0, 157.6)
- moved D1 2.32 mm to (137.2, 157.6)
- moved D33 0.54 mm to (127.5, 158.0)
- moved J1 0.10 mm to (133.0, 123.1)
Routing:
- net /VBUS: track 5.97 -> 114.7 mm, vias 0 -> 8
- net /USB_D-: track 21.7 -> 94.1 mm, vias 1 -> 4
- net /USB_D+: track 22.4 -> 94.8 mm, vias 1 -> 4
- net /VDDH: track 15.3 -> 85.9 mm, vias 2 -> 6
- net /~{nReset}: track 33.9 -> 92.5 mm, vias 6 -> 9
- net /ROW4: track 306.2 -> 340.7 mm, vias 1 -> 6
- net /ROW3: track 313.6 -> 341.2 mm, vias 2 -> 4
- net Net-(U3-P1.00/SWO): track 6.54 -> 33.2 mm, vias 1 -> 2
- net Net-(U3-SWDCLK): track 15.1 -> 37.7 mm, vias 2 -> 4
- net /COL0: track 154.9 -> 176.4 mm
- net /VDD_nRF: track 102.2 -> 123.4 mm, vias 5 -> 7
- net /ROW0: track 319.2 -> 340.1 mm, vias 1 -> 4
- net Net-(U3-SWDIO): track 13.0 -> 33.5 mm, vias 1 -> 2
- net /COL13: track 321.9 -> 342.2 mm
- net /ROW2: track 318.0 -> 332.3 mm, vias 0 -> 2
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- added copper zone on B.Cu, net /VDDH
Other:
- board text added: "Version 2.0"
- board text removed: "MX70"
- board text removed: "Version 1.0"
